Commit message: add patch to puBullet to visualize the goal

File: tamp/urdf_models/goal_patch.urdf (robot description, URDF)
Before this commit: robot green_patch, 1 links, 0 joints
Links:
- removed link green_patch
- added link goal_patch, mass 0.0; collision box size=0.0 0.0 0.0; visual box size=0.1 0.1 0.001
