Commit message: making tunnel shorter to prevent gripper collisions on pick

File: tamp/urdf_models/tunnel.urdf (robot description, URDF)
Before this commit: robot tunnel, 3 links, 2 joints
Links:
- link left_wall: geometry collision box size=0.15 0.01 0.06; visual box size=0.15 0.01 0.06
- link right_wall: geometry collision box size=0.15 0.01 0.06; visual box size=0.15 0.01 0.06
- link top_wall: geometry collision box size=0.15 0.09 0.01; visual box size=0.15 0.09 0.01
